File: UPS-MAF-APU.brd (EAGLE design)
At the start: 65 x 30 mm, 15 parts, among them J1 CONNECTOR_PI_40_PIN, J2 PJ-102AH, J3 CONNECTOR_4, J4 S4B-PH-SM4-TB(LF)(SN), J5 CONNECTOR-3, J6 CONNECTOR-6-FTDI, J7 BEL_STEWART_SI-52003-F_MAGJACK, J8 RB1-125BAG1A, U1 OLED_I2C, U2 SI7006-A20-IM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

Commit message: Add parts to schematic, change to Tabloid size page/frame.
Parts:
- removed J8: RB1-125BAG1A, APU_ENGR480_UPS_EAGLE_Library:WIZNET_RB1-125BAG1A
- J2: value PJ-102AH -> Barrel DC In
- J3: value CONNECTOR_4 -> OLED
- J4: value S4B-PH-SM4-TB(LF)(SN) -> VE.Direct Serial
- J5: value CONNECTOR-3 -> External DS18B20 Temp
- J6: value CONNECTOR-6-FTDI -> FTDI Serial Console
- J7: value BEL_STEWART_SI-52003-F_MAGJACK -> MagJack; device APU_ENGR480_UPS_EAGLE_Library:BEL_STEWART_SI-52003-F_MAGJACK -> APU_ENGR480_UPS_EAGLE_Library:WIZNET_RB1-125BAG1A
- U3: value M24C32-RDW6TP -> HAT EEPROM
- U5: value SI8621AB-B-ISR -> Isolator
- U7: value OKI-78SR-5_1.5-W36H-C -> 5V SMPS
- moved J7 30.1 mm to (-83.5, -65.5)
Changed lines of the file:
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@@
 <attribute name="NAME" x="32.5" y="15" size="2.54" layer="51" ratio="10" rot="R270" align="center"/>
 </element>
-<element name="J3" library="APU_ENGR480_UPS_EAGLE_Library" package="ESQ-104-XX-X-S" value="CONNECTOR_4" x="50.28" y="15" smashed="yes" rot="R270">
+<element name="J3" library="APU_ENGR480_UPS_EAGLE_Library" package="ESQ-104-XX-X-S" value="OLED" x="50.28" y="15" smashed="yes" rot="R270">
 <attribute name="NAME" x="53.455" y="15" size="1.524" layer="25" font="vector" ratio="10" rot="R270" align="center"/>
 <attribute name="NAME" x="50.28" y="15" size="1.524" layer="51" ratio="10" rot="R270" align="center"/>
 <attribute name="VALUE" x="47.105" y="15" size="1.524" layer="27" font="vector" ratio="10" rot="R270" align="center"/>
 </element>
-<element name="U3" library="APU_ENGR480_UPS_EAGLE_Library" package="SOP65P640X120-8N" value="M24C32-RDW6TP" x="4" y="-2.5" smashed="yes">
+<element name="U3" library="APU_ENGR480_UPS_EAGLE_Library" package="SOP65P640X120-8N" value="HAT EEPROM" x="4" y="-2.5" smashed="yes">
 <attribute name="DESCRIPTION" value="STMICROELECTRONICS - M24C32-RDW6TP - EEPROM, 32KBIT, I2C, 1MHZ, TSSOP-8" x="4" y="-2.5" size="1.778" layer="27" display="off"/>
 <attribute name="HEIGHT" value="1.2mm" x="4" y="-2.5" size="1.778" layer="27" display="off"/>
@@
 <attribute name="VALUE" x="0" y="-7.5" size="1.27" layer="27" align="center"/>
 </element>
-<element name="U7" library="APU_ENGR480_UPS_EAGLE_Library" package="OKI-78SR-HORIZONTAL" value="OKI-78SR-5_1.5-W36H-C" x="-11.5" y="-2" smashed="yes">
+<element name="U7" library="APU_ENGR480_UPS_EAGLE_Library" package="OKI-78SR-HORIZONTAL" value="5V SMPS" x="-11.5" y="-2" smashed="yes">
 <attribute name="DESCRIPTION" value="Switching Regulator 7-36Vin 5Vo 1.5A Non-Isolated DC-DC Converter, 5V dc Output, 1.5A" x="-11.5" y="-2" size="1.778" layer="27" display="off"/>
 <attribute name="HEIGHT" value="mm" x="-11.5" y="-2" size="1.778" layer="27" display="off"/>
@@
 <attribute name="VALUE" x="-11.5" y="-2" size="1.27" layer="27" align="center"/>
 </element>
-<element name="J2" library="APU_ENGR480_UPS_EAGLE_Library" package="PJ-102AH" value="PJ-102AH" x="-32" y="-5" smashed="yes">
+<element name="J2" library="APU_ENGR480_UPS_EAGLE_Library" package="PJ-102AH" value="Barrel DC In" x="-32" y="-5" smashed="yes">
 <attribute name="DESCRIPTION" value="DC POWER JACK" x="-32" y="-5" size="1.778" layer="27" display="off"/>
 <attribute name="HEIGHT" value="mm" x="-32" y="-5" size="1.778" layer="27" display="off"/>
@@
 <attribute name="VALUE" x="-30" y="-12.5" size="1.27" layer="27" align="center"/>
 </element>
-<element name="U5" library="APU_ENGR480_UPS_EAGLE_Library" package="SOIC127P600X175-8N" value="SI8621AB-B-ISR" x="-32.5" y="-17.5" smashed="yes">
+<element name="U5" library="APU_ENGR480_UPS_EAGLE_Library" package="SOIC127P600X175-8N" value="Isolator" x="-32.5" y="-17.5" smashed="yes">
 <attribute name="DESCRIPTION" value="Digital Isolators 2.5 kV 1 forward &amp; 1 reverse 2-channel isolator" x="-32.5" y="-17.5" size="1.778" layer="27" display="off"/>
 <attribute name="HEIGHT" value="1.75mm" x="-32.5" y="-17.5" size="1.778" layer="27" display="off"/>
@@
 <attribute name="VALUE" x="-32.5" y="-17.5" size="1.27" layer="27" align="center"/>
 </element>
-<element name="J5" library="APU_ENGR480_UPS_EAGLE_Library" package="MOLEX_70553-0002" value="CONNECTOR-3" x="-49.5" y="-23" smashed="yes">
+<element name="J5" library="APU_ENGR480_UPS_EAGLE_Library" package="MOLEX_70553-0002" value="External DS18B20 Temp" x="-49.5" y="-23" smashed="yes">
 <attribute name="NAME" x="-49.5" y="-23" size="1.524" layer="25" font="vector" ratio="10" align="center"/>
 <attribute name="NAME" x="-49.5" y="-23" size="2.54" layer="51" ratio="10" align="center"/>
 </element>
-<element name="J4" library="APU_ENGR480_UPS_EAGLE_Library" package="S4B-PH-SM4-TB" value="S4B-PH-SM4-TB(LF)(SN)" x="-51.5" y="-38" smashed="yes">
+<element name="J4" library="APU_ENGR480_UPS_EAGLE_Library" package="S4B-PH-SM4-TB" value="VE.Direct Serial" x="-51.5" y="-38" smashed="yes">
 <attribute name="DESCRIPTION" value="PH SMT side entry shroud header 4 way JST PH Series, 2mm Pitch 4 Way 1 Row Right Angle PCB Header, Solder Termination, 2A" x="-51.5" y="-38" size="1.778" layer="27" display="off"/>
 <attribute name="HEIGHT" value="mm" x="-51.5" y="-38" size="1.778" layer="27" display="off"/>
@@
 <attribute name="VALUE" x="-65" y="-35" size="1.27" layer="27" align="center"/>
 </element>
-<element name="J6" library="APU_ENGR480_UPS_EAGLE_Library" package="ESQ-106-XX-X-S" value="CONNECTOR-6-FTDI" x="-67.5" y="-46" smashed="yes">
+<element name="J6" library="APU_ENGR480_UPS_EAGLE_Library" package="ESQ-106-XX-X-S" value="FTDI Serial Console" x="-67.5" y="-46" smashed="yes">
 <attribute name="NAME" x="-61.15" y="-42.19" size="1.524" layer="25" font="vector" ratio="10" align="center"/>
 <attribute name="NAME" x="-61.15" y="-46" size="1.524" layer="51" ratio="10" align="center"/>
 <attribute name="VALUE" x="-61.15" y="-49.81" size="1.524" layer="27" font="vector" ratio="10" align="center"/>
 </element>
-<element name="J7" library="APU_ENGR480_UPS_EAGLE_Library" package="BEL_STEWART_SI-52003-F_MAGJACK" value="BEL_STEWART_SI-52003-F_MAGJACK" x="-81" y="-35.5" smashed="yes">
-<attribute name="NAME" x="-81" y="-21.53" size="1.27" layer="25" align="bottom-center"/>
-<attribute name="VALUE" x="-81" y="-50.105" size="1.27" layer="27" align="bottom-center"/>
-</element>
-<element name="J8" library="APU_ENGR480_UPS_EAGLE_Library" package="WIZNET_RB1-125BAG1A" value="RB1-125BAG1A" x="-83.5" y="-65.5" smashed="yes">
+<element name="J7" library="APU_ENGR480_UPS_EAGLE_Library" package="WIZNET_RB1-125BAG1A" value="MagJack" x="-83.5" y="-65.5" smashed="yes">
 <attribute name="AVAILABILITY" value="Good" x="-83.5" y="-65.5" size="1.778" layer="27" display="off"/>
 <attribute name="DESCRIPTION" value="Accessory RJ-45 With Transformer Connector - UDE" x="-83.5" y="-65.5" size="1.778" layer="27" display="off"/>

Commit message: SamChange
editpush?
Connections:
- removed net GND_1: U4.6
- removed net GND_2: U4.11
- removed net VBUS: U4.12
- removed net VS: U4.10
- new net BATTERY+: U4.12, U4.14, U4.15, U4.16
- new net BATTERY-: U4.1, U4.2, U4.3
- new net N$1: J1.8, J6.4
- new net N$2: J1.10, J6.5
- new net N$4: J1.7, J5.2
- net 3.3V: now also J5.3, J6.3, U4.10, U4.5
- net GND: now also J5.1, J6.1, U4.11, U4.4, U4.6
- net SCK: now also U2.6, U4.9
- net SDA: now also U2.1, U4.8
Changed lines of the file:
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@@
 <?xml version="1.0" encoding="utf-8"?>
 <!DOCTYPE eagle SYSTEM "eagle.dtd">
-<eagle version="9.3.1">
+<eagle version="9.3.0">
 <drawing>
 <settings>
@@
 <contactref element="J1" pad="39"/>
 <contactref element="J3" pad="1"/>
-<wire x1="50.28" y1="18.81" x2="56.63" y2="25.23" width="0" layer="19" extent="1-1"/>
-<wire x1="-31.45" y1="-12.5" x2="50.28" y2="18.81" width="0" layer="19" extent="1-1"/>
+<contactref element="J6" pad="1"/>
+<contactref element="U4" pad="4"/>
+<contactref element="U4" pad="6"/>
+<contactref element="U4" pad="11"/>
+<contactref element="J5" pad="1"/>
+<wire x1="-46.96" y1="-16.905" x2="-67.5" y2="-46" width="0" layer="19" extent="1-1"/>
+<wire x1="-31.45" y1="-12.5" x2="-46.96" y2="-16.905" width="0" layer="19" extent="1-1"/>
+<wire x1="-2.938" y1="-8.475" x2="-31.45" y2="-12.5" width="0" layer="19" extent="1-1"/>
+<wire x1="-2.938" y1="-7.175" x2="-2.938" y2="-8.475" width="0" layer="19" extent="1-1"/>
+<wire x1="2.938" y1="-8.475" x2="-2.938" y2="-8.475" width="0" layer="19" extent="1-1"/>
+<wire x1="50.28" y1="18.81" x2="2.938" y2="-8.475" width="0" layer="19" extent="1-1"/>
+<wire x1="56.63" y1="25.23" x2="50.28" y2="18.81" width="0" layer="19" extent="1-1"/>
 </signal>
 <signal name="SCLK">
@@
 <contactref element="J3" pad="3"/>
 <contactref element="J1" pad="5"/>
+<contactref element="U4" pad="9"/>
+<contactref element="U2" pad="6"/>
 <wire x1="13.45" y1="25.23" x2="50.28" y2="13.73" width="0" layer="19" extent="1-1"/>
+<wire x1="2.938" y1="-9.775" x2="13.45" y2="25.23" width="0" layer="19" extent="1-1"/>
+<wire x1="-28.55" y1="-11.5" x2="2.938" y2="-9.775" width="0" layer="19" extent="1-1"/>
 </signal>
 <signal name="SDA">
 <contactref element="J3" pad="4"/>
 <contactref element="J1" pad="3"/>
+<contactref element="U4" pad="8"/>
+<contactref element="U2" pad="1"/>
 <wire x1="10.91" y1="25.23" x2="50.28" y2="11.19" width="0" layer="19" extent="1-1"/>
-</signal>
-<signal name="GND_1">
-<contactref element="U4" pad="6"/>
-</signal>
-<signal name="VBUS">
-<contactref element="U4" pad="12"/>
-</signal>
-<signal name="GND_2">
-<contactref element="U4" pad="11"/>
-</signal>
-<signal name="VS">
-<contactref element="U4" pad="10"/>
+<wire x1="-2.938" y1="-9.775" x2="10.91" y2="25.23" width="0" layer="19" extent="1-1"/>
+<wire x1="-31.45" y1="-11.5" x2="-2.938" y2="-9.775" width="0" layer="19" extent="1-1"/>
 </signal>
 <signal name="PAD">
@@
 <contactref element="J1" pad="1"/>
 <contactref element="J3" pad="2"/>
-<wire x1="8.37" y1="25.23" x2="50.28" y2="16.27" width="0" layer="19" extent="1-1"/>
+<contactref element="J6" pad="3"/>
+<contactref element="U4" pad="5"/>
+<contactref element="U4" pad="10"/>
+<contactref element="J5" pad="3"/>
+<wire x1="-52.04" y1="-16.905" x2="-62.42" y2="-46" width="0" layer="19" extent="1-1"/>
+<wire x1="-2.938" y1="-7.825" x2="-52.04" y2="-16.905" width="0" layer="19" extent="1-1"/>
+<wire x1="2.938" y1="-9.125" x2="-2.938" y2="-7.825" width="0" layer="19" extent="1-1"/>
+<wire x1="8.37" y1="25.23" x2="2.938" y2="-9.125" width="0" layer="19" extent="1-1"/>
+<wire x1="50.28" y1="16.27" x2="8.37" y2="25.23" width="0" layer="19" extent="1-1"/>
+</signal>
+<signal name="N$1">
+<contactref element="J1" pad="8"/>
+<contactref element="J6" pad="4"/>
+<wire x1="15.99" y1="27.77" x2="-59.88" y2="-46" width="0" layer="19" extent="1-1"/>
+</signal>
+<signal name="N$2">
+<contactref element="J6" pad="5"/>
+<contactref element="J1" pad="10"/>
+<wire x1="18.53" y1="27.77" x2="-57.34" y2="-46" width="0" layer="19" extent="1-1"/>
+</signal>
+<signal name="BATTERY+">
+<contactref element="U4" pad="16"/>
+<contactref element="U4" pad="15"/>
+<contactref element="U4" pad="14"/>
+<contactref element="U4" pad="12"/>
+<wire x1="2.938" y1="-6.525" x2="2.938" y2="-7.825" width="0" layer="19" extent="1-1"/>
+<wire x1="2.938" y1="-5.875" x2="2.938" y2="-6.525" width="0" layer="19" extent="1-1"/>
+<wire x1="2.938" y1="-5.225" x2="2.938" y2="-5.875" width="0" layer="19" extent="1-1"/>
+</signal>
+<signal name="BATTERY-">
+<contactref element="U4" pad="1"/>
+<contactref element="U4" pad="3"/>
+<contactref element="U4" pad="2"/>
+<wire x1="-2.938" y1="-5.875" x2="-2.938" y2="-5.225" width="0" layer="19" extent="1-1"/>
+<wire x1="-2.938" y1="-6.525" x2="-2.938" y2="-5.875" width="0" layer="19" extent="1-1"/>
+</signal>
+<signal name="N$4">
+<contactref element="J5" pad="2"/>
+<contactref element="J1" pad="7"/>
+<wire x1="15.99" y1="25.23" x2="-49.5" y2="-16.905" width="0" layer="19" extent="1-1"/>
 </signal>
 </signals>

Commit message: README
Parts:
- added Y1: ECS-250-20-3X-EN-TR, ECS-250-20-3X-EN-TR:ECS250203XENTR
Connections:
- removed net VDDOSC: U6.25
- removed net VDDPLL: U6.20
- removed net VDDRX: U6.19
- removed net VSS: U6.2
- removed net VSSOSC: U6.22
- removed net VSSPLL: U6.21
- removed net VSSTX: U6.18
- new net N$3: U6.13
- new net N$5: U6.12
- new net N$6: J7.R2, U6.16
- new net N$7: J7.R1, U6.17
- net 3.3V: now also U6.19, U6.20, U6.25, U6.28
- net GND: now also J7.S1, J7.S2, U6.18, U6.2, U6.21, U6.22, U7.2
- net MISO: now also U6.6
- net MOSI: now also U6.7
- net SCLK: now also U6.8
- net VDD: no longer U6.28
Changed lines of the file:
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@@
 <attribute name="MF" value="WIZnet" x="-83.5" y="-65.5" size="1.778" layer="27" display="off"/>
 <attribute name="MP" value="RB1-125BAG1A" x="-83.5" y="-65.5" size="1.778" layer="27" display="off"/>
+<attribute name="NAME" x="-83.5" y="-65.5" size="5.08" layer="51" align="center"/>
 <attribute name="NAME" x="-83.500790625" y="-52.991" size="1.778" layer="25" font="vector" align="center"/>
-<attribute name="NAME" x="-83.5" y="-65.5" size="5.08" layer="51" align="center"/>
 <attribute name="PACKAGE" value="None" x="-83.5" y="-65.5" size="1.778" layer="27" display="off"/>
 <attribute name="PRICE" value="2.18 USD" x="-83.5" y="-65.5" size="1.778" layer="27" display="off"/>
+</element>
+<element name="Y1" library="ECS-250-20-3X-EN-TR" package="ECS250203XENTR" value="ECS-250-20-3X-EN-TR" x="-87.5" y="-79.5" smashed="yes">
+<attribute name="DESCRIPTION" value="CRYSTAL 25.0000MHZ 20PF SMD" x="-87.5" y="-79.5" size="1.778" layer="27" display="off"/>
+<attribute name="HEIGHT" value="2.3mm" x="-87.5" y="-79.5" size="1.778" layer="27" display="off"/>
+<attribute name="MANUFACTURER_NAME" value="ECS Inc." x="-87.5" y="-79.5" size="1.778" layer="27" display="off"/>
+<attribute name="MANUFACTURER_PART_NUMBER" value="ECS-250-20-3X-EN-TR" x="-87.5" y="-79.5" size="1.778" layer="27" display="off"/>
+<attribute name="MOUSER_PART_NUMBER" value="" x="-87.5" y="-79.5" size="1.778" layer="27" display="off"/>
+<attribute name="MOUSER_PRICE-STOCK" value="" x="-87.5" y="-79.5" size="1.778" layer="27" display="off"/>
+<attribute name="NAME" x="-87.5" y="-79.5" size="1.27" layer="25" align="center"/>
+<attribute name="RS_PART_NUMBER" value="" x="-87.5" y="-79.5" size="1.778" layer="27" display="off"/>
+<attribute name="RS_PRICE-STOCK" value="" x="-87.5" y="-79.5" size="1.778" layer="27" display="off"/>
+<attribute name="VALUE" x="-87.5" y="-79.5" size="1.27" layer="27" align="center"/>
 </element>
 </elements>
@@
 <signal name="MOSI">
 <contactref element="J1" pad="19"/>
+<contactref element="U6" pad="7"/>
+<wire x1="31.23" y1="25.23" x2="-68.55" y2="-34.675" width="0" layer="19" extent="1-1"/>
 </signal>
 <signal name="GND">
@@
 <contactref element="U4" pad="11"/>
 <contactref element="J5" pad="1"/>
-<wire x1="-46.96" y1="-16.905" x2="-67.5" y2="-46" width="0" layer="19" extent="1-1"/>
+<contactref element="J7" pad="S2"/>
+<contactref element="J7" pad="S1"/>
+<contactref element="U6" pad="2"/>
+<contactref element="U6" pad="22"/>
+<contactref element="U6" pad="21"/>
+<contactref element="U6" pad="18"/>
+<contactref element="U7" pad="2"/>
+<wire x1="-75.625790625" y1="-62.451040625" x2="-91.375790625" y2="-62.451040625" width="0" layer="19" extent="1-1"/>
+<wire x1="-67.5" y1="-46" x2="-75.625790625" y2="-62.451040625" width="0" layer="19" extent="1-1"/>
+<wire x1="-61.45" y1="-37.275" x2="-67.5" y2="-46" width="0" layer="19" extent="1-1"/>
+<wire x1="-61.45" y1="-35.325" x2="-61.45" y2="-37.275" width="0" layer="19" extent="1-1"/>
+<wire x1="-61.45" y1="-34.675" x2="-61.45" y2="-35.325" width="0" layer="19" extent="1-1"/>
+<wire x1="-68.55" y1="-31.425" x2="-61.45" y2="-34.675" width="0" layer="19" extent="1-1"/>
+<wire x1="-46.96" y1="-16.905" x2="-61.45" y2="-34.675" width="0" layer="19" extent="1-1"/>
 <wire x1="-31.45" y1="-12.5" x2="-46.96" y2="-16.905" width="0" layer="19" extent="1-1"/>
-<wire x1="-2.938" y1="-8.475" x2="-31.45" y2="-12.5" width="0" layer="19" extent="1-1"/>
+<wire x1="-11.5" y1="-8.95" x2="-31.45" y2="-12.5" width="0" layer="19" extent="1-1"/>
+<wire x1="-2.938" y1="-8.475" x2="-11.5" y2="-8.95" width="0" layer="19" extent="1-1"/>
 <wire x1="-2.938" y1="-7.175" x2="-2.938" y2="-8.475" width="0" layer="19" extent="1-1"/>
 <wire x1="2.938" y1="-8.475" x2="-2.938" y2="-8.475" width="0" layer="19" extent="1-1"/>
@@
 <signal name="SCLK">
 <contactref element="J1" pad="23"/>
+<contactref element="U6" pad="8"/>
+<wire x1="36.31" y1="25.23" x2="-68.55" y2="-35.325" width="0" layer="19" extent="1-1"/>
 </signal>
 <signal name="MISO">
 <contactref element="J1" pad="21"/>
+<contactref element="U6" pad="6"/>
+<wire x1="33.77" y1="25.23" x2="-68.55" y2="-34.025" width="0" layer="19" extent="1-1"/>
 </signal>
 <signal name="SCK">
@@
 <signal name="VDD">
 <contactref element="U2" pad="5"/>
-<contactref element="U6" pad="28"/>
-<wire x1="-28.55" y1="-12.5" x2="-61.45" y2="-30.775" width="0" layer="19" extent="1-1"/>
-</signal>
-<signal name="VSS">
-<contactref element="U6" pad="2"/>
 </signal>
 <signal name="VSSRX">
 <contactref element="U6" pad="11"/>
-</signal>
-<signal name="VDDOSC">
-<contactref element="U6" pad="25"/>
-</signal>
-<signal name="VSSOSC">
-<contactref element="U6" pad="22"/>
-</signal>
-<signal name="VSSPLL">
-<contactref element="U6" pad="21"/>
-</signal>
-<signal name="VDDPLL">
-<contactref element="U6" pad="20"/>
-</signal>
-<signal name="VDDRX">
-<contactref element="U6" pad="19"/>
-</signal>
-<signal name="VSSTX">
-<contactref element="U6" pad="18"/>
 </signal>
 <signal name="VDDTX">
@@
 <contactref element="U4" pad="10"/>
 <contactref element="J5" pad="3"/>
-<wire x1="-52.04" y1="-16.905" x2="-62.42" y2="-46" width="0" layer="19" extent="1-1"/>
+<contactref element="U6" pad="28"/>
+<contactref element="U6" pad="25"/>
+<contactref element="U6" pad="20"/>
+<contactref element="U6" pad="19"/>
+<wire x1="-61.45" y1="-36.625" x2="-62.42" y2="-46" width="0" layer="19" extent="1-1"/>
+<wire x1="-61.45" y1="-35.975" x2="-61.45" y2="-36.625" width="0" layer="19" extent="1-1"/>
+<wire x1="-61.45" y1="-32.725" x2="-61.45" y2="-35.975" width="0" layer="19" extent="1-1"/>
+<wire x1="-61.45" y1="-30.775" x2="-61.45" y2="-32.725" width="0" layer="19" extent="1-1"/>
+<wire x1="-52.04" y1="-16.905" x2="-61.45" y2="-30.775" width="0" layer="19" extent="1-1"/>
 <wire x1="-2.938" y1="-7.825" x2="-52.04" y2="-16.905" width="0" layer="19" extent="1-1"/>
 <wire x1="2.938" y1="-9.125" x2="-2.938" y2="-7.825" width="0" layer="19" extent="1-1"/>
@@
 <wire x1="15.99" y1="25.23" x2="-49.5" y2="-16.905" width="0" layer="19" extent="1-1"/>
 </signal>
+<signal name="N$3">
+<contactref element="U6" pad="13"/>
+</signal>
+<signal name="N$5">
+<contactref element="U6" pad="12"/>
+</signal>
+<signal name="N$6">
+<contactref element="J7" pad="R2"/>
+<contactref element="U6" pad="16"/>
+<wire x1="-61.45" y1="-38.575" x2="-86.675790625" y2="-56.611040625" width="0" layer="19" extent="1-1"/>
+</signal>
+<signal name="N$7">
+<contactref element="J7" pad="R1"/>
+<contactref element="U6" pad="17"/>
+<wire x1="-61.45" y1="-37.925" x2="-87.945790625" y2="-59.151040625" width="0" layer="19" extent="1-1"/>
+</signal>
 </signals>
